File: hardware-design/road-marking-robot-circuits/_autosave-road-marking-robot-circuits.kicad_sch (KiCad schematic)
At the start: 73 parts, among them J1 DC Barrel Jack THT, J10 2 PIN terminal Block, J11 2PIN terminal block, J12 2PIN terminal block, J13 2PIN terminal block, J14 MOTOR_DRIVER, J2 u-sonic-1, J3 u-sonic-2, J4 u-sonic-3, J5 u-sonic-4, J6 u-sonic-5, J7 3PIN Terminal block, J8 2PIN terminal block, J9 2 pin Terminal block, K1 SugarCube relay, K2 SugarCube relay, K3 SugarCube relay, K4 SugarCube relay, M2 ROBOT_WHEEL, Q1 BC547 transistor, Q2 BC547 transistor, Q3 BC547 transistor, Q4 BC547 transistor, SW1 2pin terminal block, SW2 push button pin, U1 LM7909_TO220, U2 LM7812_TO220, U3 LM7805_TO220, U4 LM7806_TO220, U5 NE06M GPS Module, U6 L293D Motor driver chip

Commit message: updates FIRMWARE for ARDUINO
Connections:
- net 12V_UNREG: now also J8.1 (Pin_1)
- net Earth: now also K1.11
Changed lines of the file:
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@@
 	(wire
 		(pts
-			(xy 198.12 209.55) (xy 198.12 203.2)
+			(xy 191.77 203.2) (xy 191.77 198.12)
 		)
 		(stroke
@@
 	(wire
 		(pts
-			(xy 198.12 203.2) (xy 210.82 203.2)
-		)
-		(stroke
-			(width 0)
-			(type default)
-		)
-	)
-	(wire
-		(pts
 			(xy 297.18 269.24) (xy 311.15 269.24)
 		)
@@
 	(wire
 		(pts
+			(xy 210.82 201.93) (xy 210.82 203.2)
+		)
+		(stroke
+			(width 0)
+			(type default)
+		)
+	)
+	(wire
+		(pts
 			(xy 184.15 292.1) (xy 184.15 289.56)
 		)
@@
 	(wire
 		(pts
+			(xy 198.12 203.2) (xy 198.12 209.55)
+		)
+		(stroke
+			(width 0)
+			(type default)
+		)
+	)
+	(wire
+		(pts
 			(xy 257.81 220.98) (xy 261.62 220.98)
 		)
@@
 	(wire
 		(pts
+			(xy 191.77 203.2) (xy 198.12 203.2)
+		)
+		(stroke
+			(width 0)
+			(type default)
+		)
+	)
+	(wire
+		(pts
 			(xy 232.41 128.27) (xy 234.95 128.27)
 		)
@@
 	(text "SOLENOID RELAY\n"
 		(exclude_from_sim no)
-		(at 199.136 200.914 0)
+		(at 184.912 192.278 0)
 		(effects
 			(font
@@
 		)
 	)
-	(text "*NO to prevent\nleakage on boot\n"
-		(exclude_from_sim no)
-		(at 203.708 222.504 0)
-		(effects
-			(font
-				(size 1.27 1.27)
-			)
-		)
-	)
 	(text "SPRAY GUN RELAY"
 		(exclude_from_sim no)
@@
 		)
 	)
+	(global_label "12V_UNREG"
+		(shape input)
+		(at 191.77 198.12 180)
+		(fields_autoplaced yes)
+		(effects
+			(font
+				(size 1.27 1.27)
+			)
+			(justify right)
+		)
+		(property "Intersheetrefs" "${INTERSHEET_REFS}"
+			(at 179.2549 198.12 0)
+			(effects
+				(font
+					(size 1.27 1.27)
+				)
+				(justify right)
+				(hide yes)
+			)
+		)
+	)
 	(global_label "6V_REG"
 		(shape input)
@@
 		(length 2.54)
 		(shape dot)
-		(at 200.66 203.2 0)
-		(fields_autoplaced yes)
-		(effects
-			(font
-				(size 1.27 1.27)
-			)
-			(justify left bottom)
-		)
-		(property "Netclass" "power"
-			(at 201.3585 200.66 0)
-			(show_name yes)
-			(effects
-				(font
-					(size 1.27 1.27)
-					(italic yes)
-				)
-				(justify left)
-			)
-		)
-	)
-	(netclass_flag ""
-		(length 2.54)
-		(shape dot)
 		(at 149.86 143.51 0)
 		(fields_autoplaced yes)
@@
 	)
 	(symbol
+		(lib_id "power:Earth")
+		(at 210.82 201.93 180)
+		(unit 1)
+		(exclude_from_sim no)
+		(in_bom yes)
+		(on_board yes)
+		(dnp no)
+		(fields_autoplaced yes)
+		(property "Reference" "#PWR037"
+			(at 210.82 195.58 0)
+			(effects
+				(font
+					(size 1.27 1.27)
+				)
+				(hide yes)
+			)
+		)
+		(property "Value" "Earth"
+			(at 210.82 196.85 0)
+			(effects
+				(font
+					(size 1.27 1.27)
+				)
+				(hide yes)
+			)
+		)
+		(property "Footprint" ""
+			(at 210.82 201.93 0)
+			(effects
+				(font
+					(size 1.27 1.27)
+				)
+				(hide yes)
+			)
+		)
+		(property "Datasheet" "~"
+			(at 210.82 201.93 0)
+			(effects
+				(font
+					(size 1.27 1.27)
+				)
+				(hide yes)
+			)
+		)
+		(property "Description" "Power symbol creates a global label with name \"Earth\""
+			(at 210.82 201.93 0)
+			(effects
+				(font
+					(size 1.27 1.27)
+				)
+				(hide yes)
+			)
+		)
+		(pin "1"
+		)
+		(instances
+			(project "road-marking-robot-circuits"
+				(path "/95faade6-3887-4eb7-bcc3-fce13ba0f784"
+					(reference "#PWR037")
+					(unit 1)
+				)
+			)
+		)
+	)
+	(symbol
 		(lib_id "Diode:1N4001")
 		(at 229.87 210.82 270)
@@
 		(dnp no)
 		(property "Reference" "J8"
-			(at 193.675 204.47 0)
+			(at 183.896 204.724 0)
 			(effects
 				(font
@@
 		)
 		(property "Value" "2PIN terminal block"
-			(at 191.008 207.01 0)
+			(at 189.484 207.01 0)
 			(effects
 				(font
